Commit message: considering panda now

File: lite-6-sim-teleop/lite-6-updated-urdf/lite_6_gripper.urdf (robot description, URDF)
Before this commit: robot gripper_model, 3 links, 2 joints
Joints:
- joint left_finger_joint: axis (none) -> 1 0 0; limit (none) -> lower=0.0 upper=0.04 effort=120 velocity=0.1; origin (none) -> xyz=0 0 0 rpy=0 0 0; type fixed -> prismatic
- joint right_finger_joint: axis (none) -> -1 0 0; limit (none) -> lower=0.0 upper=0.04 effort=120 velocity=0.1; origin (none) -> xyz=0 0 0 rpy=0 0 0; type fixed -> prismatic
